File: HW/Breakout_FDC2212/Breakout_FDC2212.kicad_pcb (KiCad board)
At the start: 2 copper layers, 26 x 18 mm, 21 parts, among them J1 SM04B-SRSS-TB, J2 Conn_01x02, J3 Conn_01x02, J4 Conn_01x06, U5 625L3C040M00000, U6 FDC2212

Commit message: FDC2212v2
Parts:
- removed the C3 at (108.0, 112.5)
- removed the R1 at (108.0, 103.5)
- removed R7, R8: 10k, Resistor_SMD:R_0603_1608Metric
- added JP1: Jumper_IN0B, Jumper:SolderJumper-2_P1.3mm_Bridged_RoundedPad1.0x1.5mm, F.Cu at (117.8, 106.2)
- added R2: 10k, Resistor_SMD:R_0603_1608Metric, F.Cu at (110.9, 101.7)
- added R3: 10k, Resistor_SMD:R_0603_1608Metric, F.Cu at (110.9, 103.3)
- added R4: 100k, Resistor_SMD:R_0603_1608Metric, F.Cu at (107.9, 103.3)
- added R5: 100k, Resistor_SMD:R_0603_1608Metric, F.Cu at (109.6, 112.4)
- C2, C4: footprint Capacitor_SMD:C_0603_1608Metric -> Capacitor_SMD:C_0402_1005Metric
- J1: value SM04B-SRSS-TB -> Conn_Qwiic
- J2, J3: footprint Connector_PinHeader_2.54mm:PinHeader_1x02_P2.54mm_Vertical -> Connector_PinHeader_2.54mm:PinHeader_1x03_P2.54mm_Vertical
- J4: value Conn_01x06 -> Conn_Breadboard
- R1: renamed from R4; value 680 -> 4.7k
- moved C2 3.90 mm to (115.4, 112.4), turned to 0 degrees
- moved J3 2.54 mm to (114.3, 102.8)
- moved C1 2.18 mm to (112.8, 112.4), turned to 180 degrees
- moved C3 1.41 mm to (118.4, 109.2)
- moved J2 1.41 mm to (124.2, 106.5)
- moved C4 1.29 mm to (109.0, 106.3), turned to 90 degrees
- moved L1 1.13 mm to (120.8, 109.8)
- moved R1 0.24 mm to (107.9, 101.7)
- moved H1 0.10 mm to (102.5, 102.6)
- renumbered C13 to C3, D3 to D1, U5 to U1, U6 to U2
Connections:
- U2 pad 10: /SENSE0- -> Net-(JP1-A)
Routing:
- net Net-(JP1-A): track 0.00 -> 4.23 mm
- net /SENSE0+: track 9.13 -> 11.3 mm
- net /SENSE1+: track 8.44 -> 6.50 mm
- net +3.3V: track 41.0 -> 42.3 mm
- net /SDA: track 38.1 -> 37.1 mm
- net /SCL: track 41.4 -> 40.8 mm
- net /FDC_SHUTDOWN: track 12.9 -> 13.5 mm
- net /SENSE1-: track 5.74 -> 5.21 mm
- net GND: track 2.18 -> 2.35 mm, vias 51 -> 37
Other:
- board size 26 x 18 mm -> 26 x 17.9 mm
- board text added: "0A"
- board text added: "0B"
- board text added: "1A"
- board text added: "1B"
- board text added: "FDC2212 Breakout Capacitance-to-digital converter 28-bit resolution, L-C tank I2C address 0x2A Daniel Stiner ${REVISION}"
- board text added: "JMP_0B"
- board text removed: "FDC2212 Breakout Capacitance-to-digital converter 28-bit resolution, L-C tank I2C address 0x2A Daniel Stiner 2025v0.2"
