File: HW/Breakout_FDC2212/Breakout_FDC2212.kicad_sch (KiCad schematic)
At the start: 21 parts, among them J1 Conn_Qwiic, J2 Conn_01x02, J3 Conn_01x02, J4 Conn_Breadboard, U5 625L3C040M00000, U6 FDC2212

Commit message: FDC2212v2
Parts:
- removed C3: 0.01u, Capacitor_SMD:C_0603_1608Metric, symbol Device:C
- removed R1, R7, R8: 10k, Resistor_SMD:R_0603_1608Metric, symbol Device:R
- added JP1: Jumper_IN0B, Jumper:SolderJumper-2_P1.3mm_Bridged_RoundedPad1.0x1.5mm, symbol Jumper:SolderJumper_2_Bridged
- added R2, R3: 10k, Resistor_SMD:R_0603_1608Metric, symbol Device:R
- added R4, R5: 100k, Resistor_SMD:R_0603_1608Metric, symbol Device:R
- C2, C4: footprint Capacitor_SMD:C_0603_1608Metric -> Capacitor_SMD:C_0402_1005Metric
- J2, J3: footprint Connector_PinHeader_2.54mm:PinHeader_1x02_P2.54mm_Vertical -> Connector_PinHeader_2.54mm:PinHeader_1x03_P2.54mm_Vertical; symbol Connector_Generic:Conn_01x02 -> Connector_Generic:Conn_01x03
- R1: renamed from R4; value 680 -> 4.7k
- renumbered C13 to C3, D3 to D1, U5 to U1, U6 to U2
Connections:
- net +3.3V: now also R2.1, R3.1, R4.1
- net EOH: now also R4.2
- net FDC_SHUTDOWN: now also R5.1
- net GND: now also J2.3 (Pin_3), J3.3 (Pin_3), R5.2
- net SCL: now also R3.2
- net SDA: now also R2.2
- net SENSE0-: now also JP1.2 (B); no longer U2.10 (IN0B)
- new net: JP1.1 (A), U2.10 (IN0B)
Other:
- title: Breakout  for FDC2212 Capacitance-to-Digital -> Breakout  for FDC2212 Capacitance-to-Digital Converter
- moved on the sheet: C3, J1, L1
