File: HW/Breakout_FDC1004/Breakout_FDC1004.kicad_pcb (KiCad board)
At the start: 2 copper layers, 26 x 18 mm, 14 parts, among them J1 Conn_Qwiic, J3 Conn_CIN2, J4 Conn_Breadboard, U6 FDC1004DSCR

Commit message: v1 FDC1004 breakout
Parts:
- R1: renamed from R4; value 1k -> 4.7k
- U1: renamed from U6; value FDC1004DSCR -> FDC1004
- moved R3 18.5 mm to (112.4, 112.8)
- moved R2 16.8 mm to (109.1, 112.8)
- moved C2 15.0 mm to (107.6, 108.9), turned to 90 degrees
- moved C1 14.6 mm to (107.4, 105.9), turned to -90 degrees
- moved R1 0.10 mm to (107.4, 102.6)
- moved U1 0.08 mm to (111.0, 109.5)
- renumbered D3 to D1, R7 to R2, R8 to R3
Connections:
- J3 pad 1: unconnected-(J3-Pin_1-Pad1) -> GND
- J3 pad 3: unconnected-(J3-Pin_3-Pad3) -> /SHLD1
- U1 pad V: (no net) -> GND
Routing:
- net +3.3V: track 17.4 -> 33.3 mm
- net /CIN2: track 0.00 -> 12.1 mm
- net /CIN1: track 0.00 -> 10.4 mm
- net /CIN3: track 0.00 -> 8.22 mm
- net /SDA: track 19.2 -> 26.3 mm, vias 1 -> 2
- net /SHLD2: track 0.00 -> 5.62 mm, vias 0 -> 4
- net GND: track 0.85 -> 5.57 mm, vias 9 -> 11
- net /CIN4: track 0.00 -> 4.42 mm
- net /SHLD1: track 0.00 -> 3.40 mm, vias 0 -> 3
- net /SCL: track 26.2 -> 29.1 mm
- net Net-(D1-A): track 0.30 -> 1.92 mm
Other:
- board text added: "CIN1"
- board text added: "CIN2"
- board text added: "CIN3 SHLD2"
- board text added: "FDC1004 Breakout Capacitance-to-digital converter 0.5fF resolution over ±15pF range Max 100pF offset, 400pF shield I2C address 0x50 Daniel Stiner ${REVISION}"
- board text added: "SHLD1"
- board text removed: "CIN3 SHLD1"
- board text removed: "FDC2112 Breakout Capacitance-to-digital converter 16-bit resolution, L-C tank I2C address 0x2A Daniel Stiner 2025v0.1"
