File: HW/Breakout_FDC1004/Breakout_FDC1004.kicad_sch (KiCad schematic)
At the start: 21 parts, among them J1 Conn_Qwiic, J2 Conn_01x02, J3 Conn_01x02, J4 Conn_Breadboard, U5 625L3C040M00000, U6 FDC2212

Commit message: FDC1004 progress and misc cleanup
Parts:
- removed C13: 33p, Capacitor_SMD:C_0603_1608Metric, symbol Device:C
- removed C3: 0.01u, Capacitor_SMD:C_0603_1608Metric, symbol Device:C
- removed C4: 0.1u, Capacitor_SMD:C_0603_1608Metric, symbol Device:C
- removed J2: Conn_01x02, Connector_PinHeader_2.54mm:PinHeader_1x02_P2.54mm_Vertical, symbol Connector_Generic:Conn_01x02
- removed L1: 10uH, Inductor_SMD:L_1210_3225Metric, symbol Device:L_Iron
- removed R1: 10k, Resistor_SMD:R_0603_1608Metric, symbol Device:R
- removed U5: 625L3C040M00000, 625L3C040M00000:IC_625L3C040M00000_CTS, symbol 625L3C040M00000:625L3C040M00000
- C2: footprint Capacitor_SMD:C_0603_1608Metric -> Capacitor_SMD:C_0402_1005Metric; Digikey Part Number 490-5798-1-ND -> (none)
- J3: value Conn_01x02 -> Conn_CIN2; footprint Connector_PinHeader_2.54mm:PinHeader_1x02_P2.54mm_Vertical -> Connector_PinHeader_2.54mm:PinHeader_1x03_P2.54mm_Vertical; symbol Connector_Generic:Conn_01x02 -> Connector_Generic:Conn_01x03
- R4: value 680 -> 1k
- U6: value FDC2212 -> FDC1004DSCR; footprint FDC2212DNTT:DNT0012B -> FDC1004DSCR:DSC0010B; symbol FDC2212DNTR:FDC2212DNTR -> FDC1004DSCR:FDC1004DSCR; Digikey Part Number 296-42304-1-ND -> 296-44560-1-ND; Part Number FDC2212DNTT -> FDC2112QDNTRQ1
Connections:
- net SENSE0+ is gone; now on net SCL: U6.9 (SCL)
- net SENSE0- is gone; now on net SDA: U6.10 (SDA)
- net +3.3V: now also U6.8 (VDD); no longer U6.7 (VDD)
- net GND: now also U6.11 (DAP), U6.7 (GND); no longer U6.13 (PAD), U6.4 (ADDR), U6.8 (GND), U6.V (VIA)
- net SCL: no longer U6.1 (SCL)
- net SDA: no longer U6.2 (SDA)
- net CIN4: now reaches U6.5 (CIN4)
- net EOH renamed SHLD1
- net SHLD1: now also U6.1 (SHLD1)
- net FDC_CLK renamed CIN2
- net CIN2: now also J3.2 (Pin_2)
- net FDC_SHUTDOWN renamed CIN1
- net CIN1: now also U6.2 (CIN1); no longer U6.6 (SD)
- removed net SENSE1+: J3.2 (Pin_2), U6.11 (IN1A)
- net SENSE1-: no longer names the net of J3.1 (Pin_1)
- net SENSE1-: no longer U6.12 (IN1B)
- new net CIN3: U6.4 (CIN3)
- new net SHLD2: U6.6 (SHLD2)
- no-connect marks 1 -> 0
Other:
- note removed: "I2C Address 0x2A"
- note removed: "L-C Tank C2D Sensor"
- title: Breakout  for FDC2212 Capacitance-to-Digital -> FDC1004 Capacitance-to-Digital Converter Breakout
- moved on the sheet: C1, C2, D3, J1, J4, R4

Commit message: v1 FDC1004 breakout
Parts:
- R1: renamed from R4; value 1k -> 4.7k
- U1: renamed from U6; value FDC1004DSCR -> FDC1004; Digikey Part Number 296-44560-1-ND -> (none); Part Number FDC2112QDNTRQ1 -> (none)
- renumbered D3 to D1, R7 to R2, R8 to R3
Connections:
- net GND: now also J3.1 (Pin_1), U1.V (VIA)
- net SHLD1: now also J3.3 (Pin_3)
Other:
- moved on the sheet: J3
