File: HW/Breakout_BQ25570_Cap/Breakout_BQ25570_Cap.kicad_pcb (KiCad board)
At the start: 2 copper layers, 32 x 26 mm, 42 parts, among them J1 Conn_Breadboard, J2 BAT_EXTRA, SW1 Test, U1 BQ25570

Commit message: FDC1004 progress and misc cleanup
Other:
- board text added: "${TITLE} Ultra low power, min 600mV cold start Input: Two BPW34 photodiodes in series Storage: Peak 5.5V, parallel 100uF MLCCs Output: 3.3V, peak 110mA Bridge ~{EN} to GND to enable charging Bridge VOK to OUTEN to enable output Bridge VIN to BPW to use onboard BPW34's Output requires VBAT>3.5V with 4.5V hysteresis"
- board text added: "Daniel Stiner ${REVISION}"
- board text removed: "BQ25570 Solar Harvester Breakout Ultra low power, min 600mV cold start Input: Two BPW34 photodiodes in series Storage: Peak 5.5V, parallel 100uF MLCCs Output: 3.3V, peak 110mA Bridge ~{EN} to GND to enable charging Bridge VOK to OUTEN to enable output Bridge VIN to BPW to use onboard BPW34's Output requires VBAT>3.5V with 4.5V hysteresis"
- board text removed: "Daniel Stiner 2025v0.1"
Changed lines of the file:
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@@
 		)
 	)
+	(property "REVISION" "2")
+	(property "YEAR" "2025")
 	(net 0 "")
 	(net 1 "/VIN")
@@
 		)
 	)
-	(gr_text "Daniel Stiner 2025v0.1"
+	(gr_text "Daniel Stiner ${REVISION}"
 		(at 120 118 0)
 		(layer "B.SilkS")
@@
 		)
 	)
-	(gr_text "BQ25570 Solar Harvester Breakout\nUltra low power, min 600mV cold start\n\nInput: Two BPW34 photodiodes in series\nStorage: Peak 5.5V, parallel 100uF MLCCs\nOutput: 3.3V, peak 110mA\n\nBridge ~{EN} to GND to enable charging\nBridge VOK to OUTEN to enable output\nBridge VIN to BPW to use onboard BPW34's\nOutput requires VBAT>3.5V with 4.5V hysteresis"
+	(gr_text "${TITLE}\nUltra low power, min 600mV cold start\n\nInput: Two BPW34 photodiodes in series\nStorage: Peak 5.5V, parallel 100uF MLCCs\nOutput: 3.3V, peak 110mA\n\nBridge ~{EN} to GND to enable charging\nBridge VOK to OUTEN to enable output\nBridge VIN to BPW to use onboard BPW34's\nOutput requires VBAT>3.5V with 4.5V hysteresis"
 		(at 128.2 116.4 0)
 		(layer "B.SilkS")

Commit message: BQ25570 breakout v2
- 1.8V output
- Aligned headers for breadboarding
Parts:
- added C_BAT6: 100u, Capacitor_SMD:C_1206_3216Metric, B.Cu at (126.5, 107.1)
- COUT1: value 4.7u -> 47u; footprint Capacitor_SMD:C_0805_2012Metric -> Capacitor_SMD:C_0603_1608Metric
- C_BAT1, C_BAT2, TP2, TP3: moved to B.Cu
- J1: footprint Connector_PinHeader_2.54mm:PinHeader_1x05_P2.54mm_Vertical -> Connector_PinHeader_2.54mm:PinHeader_1x06_P2.54mm_Vertical
- J2: value BAT_EXTRA -> EXCAP; footprint Connector_PinHeader_2.54mm:PinHeader_1x02_P2.54mm_Vertical -> Connector_PinHeader_2.54mm:PinHeader_1x03_P2.54mm_Vertical
- R4: value 1k -> 2k
- ROK1: value 3.57M -> 3.57M 1%
- ROK2: value 6.80M -> 2.32M 1%
- ROK3: value 3.00M -> 7.50M 1%
- ROV1: value 4.32M -> 4.32M 1%
- ROV2: value 8.66M -> 8.66M 1%
- RVO1: value 4.70M -> 8.66M 1%
- RVO2: value 7.87M -> 4.32M 1%
- moved C_BAT1 10.7 mm to (126.5, 102.1), turned to 0 degrees
- moved C_BAT2 9.67 mm to (126.5, 104.6), turned to 0 degrees
- moved TP4 7.83 mm to (121.7, 102.0)
- moved J2 7.01 mm to (115.5, 99.2), turned to 90 degrees
- moved J3 1.81 mm to (105.4, 99.2)
- moved TP3 0.64 mm to (113.3, 100.1), turned to 180 degrees
- moved TP2 0.42 mm to (111.2, 100.9), turned to 180 degrees
- renumbered JP1 to J3
Connections:
- C_BAT1 pad 1: /VBAT -> Net-(J2-Pin_3)
- C_BAT2 pad 1: /VBAT -> Net-(J2-Pin_3)
- C_BAT3 pad 1: /VBAT -> Net-(J2-Pin_3)
- C_BAT4 pad 1: /VBAT -> Net-(J2-Pin_3)
- C_BAT5 pad 1: /VBAT -> Net-(J2-Pin_3)
- J2 pad 1: /VBAT -> GND
- J2 pad 2: GND -> /VBAT
Routing:
- net Net-(J2-Pin_3): track 0.00 -> 20.1 mm, vias 0 -> 3
- net /VBAT: track 27.0 -> 16.3 mm
- net Net-(D1-A): track 5.51 -> 6.91 mm
- net /VSTOR: track 31.0 -> 32.1 mm, vias 2 -> 3
- net VOUT: track 21.3 -> 20.6 mm
- net /LBOOST: track 8.23 -> 8.29 mm, vias 0 -> 1
- net GND: vias 63 -> 62
Other:
- board text added: "${TITLE} Ultra low power, min 600mV cold start Input: Two BPW34 photodiodes (or external) Storage: Peak 5.5V, parallel 1206 MLCCs Output: 1.8V, peak 110mA"
- board text added: "Bridge ~{EN} to GND to enable charging Bridge VOK to OUTEN to enable output Bridge VIN to BPW to use onboard BPW34's Bridge VBAT to CAP to use onboard MLCC's VOK requires VBAT>2.0V with 4.5V hysteresis"
- board text added: "CAP"
- board text removed: "${TITLE} Ultra low power, min 600mV cold start Input: Two BPW34 photodiodes in series Storage: Peak 5.5V, parallel 100uF MLCCs Output: 3.3V, peak 110mA Bridge ~{EN} to GND to enable charging Bridge VOK to OUTEN to enable output Bridge VIN to BPW to use onboard BPW34's Output requires VBAT>3.5V with 4.5V hysteresis"
