File: HW/Breakout_BQ25570_Cap/Breakout_BQ25570_Cap.kicad_sch (KiCad schematic)
At the start: 42 parts, among them J1 Conn_Breadboard, J2 BAT_EXTRA, SW1 Test, U1 BQ25570

Commit message: FDC1004 progress and misc cleanup
Parts:
- added R1, R2: 100k, symbol Device:R
- ROK1: value 3.57M -> 3.57M 1%
- ROK2: value 6.80M -> 6.80M 1%
- ROV1: value 4.32M -> 4.32M 1%
- ROV2: value 8.66M -> 8.66M 1%
- RVO1: value 4.70M -> 4.70M 1%
- RVO2: value 7.87M -> 7.87M 1%
Connections:
- net GND: now also R2.2
- net VOUT_EN: now also R2.1
- net VSTOR: now also R1.1
- net ~{EN}: now also R1.2
Other:
- note added: "Defaults to disabled"
- title: Breakout for BQ25570 Energy Harvester -> BQ25570 Solar Harvester Breakout
- moved on the sheet: CREF1

Commit message: BQ25570 breakout v2
- 1.8V output
- Aligned headers for breadboarding
Parts:
- removed R1, R2: 100k, symbol Device:R
- added C_BAT6: 100u, Capacitor_SMD:C_1206_3216Metric, symbol Device:C
- COUT1: value 4.7u -> 47u; footprint Capacitor_SMD:C_0805_2012Metric -> Capacitor_SMD:C_0603_1608Metric
- CREF1: Digikey Part Number (none) -> 1276-1028-1-ND
- J1: footprint Connector_PinHeader_2.54mm:PinHeader_1x05_P2.54mm_Vertical -> Connector_PinHeader_2.54mm:PinHeader_1x06_P2.54mm_Vertical; symbol Connector_Generic:Conn_01x05 -> Connector_Generic:Conn_01x06
- J2: value BAT_EXTRA -> EXCAP; footprint Connector_PinHeader_2.54mm:PinHeader_1x02_P2.54mm_Vertical -> Connector_PinHeader_2.54mm:PinHeader_1x03_P2.54mm_Vertical; symbol Connector_Generic:Conn_01x02 -> Connector_Generic:Conn_01x03
- R4: value 1k -> 2k
- ROK2: value 6.80M 1% -> 2.32M 1%
- ROK3: value 3.00M -> 7.50M 1%
- RVO1: value 4.70M 1% -> 8.66M 1%
- RVO2: value 7.87M 1% -> 4.32M 1%
- renumbered JP1 to J3
Connections:
- net GND: now also J1.6 (Pin_6), J2.1 (Pin_1), C_BAT6.2; no longer J2.2 (Pin_2)
- net VBAT: now also J2.2 (Pin_2); no longer C_BAT1.1, C_BAT2.1, C_BAT3.1, C_BAT4.1, C_BAT5.1, J2.1 (Pin_1)
- new net: C_BAT1.1, C_BAT2.1, C_BAT3.1, C_BAT4.1, C_BAT5.1, C_BAT6.1, J2.3 (Pin_3)
Other:
- note added: "1.8V"
- note added: "2.0V"
- note added: "Enable charging by bridging ~{EN} to GND Enable output by bridging VOUT_EN to VBAT_OK Connect load between VOUT and GND Peak output 110mA@1.8V"
- note added: "Storage maximized by setting VBAT_OV to maximum supported voltage. Output voltage 1.8V with 200mV dropout allowance. See design help spreadsheet for calculations"
- note removed: "3.3V"
- note removed: "3.5V"
- note removed: "Enable charging by bridging ~{EN} to GND Enable output by bridging VOUT_EN to VBAT_OK Connect load between VOUT and GND Peak output 110mA@3.3V"
- note removed: "Storage maximized by setting VBAT_OV to maximum supported voltage. Output voltage 3.3V with 200mV dropout allowance. See design help spreadsheet for calculations"
